Commit message: data

File: urdf_publisher/urdf/humanSubject01_48dof.urdf (robot description, URDF)
Before this commit: robot XSensStyleModel_template, 52 links, 51 joints
Joints:
- joint human_location: origin xyz=0           0    0 rpy=0 0 3.14 -> xyz=0           0    0 rpy=0 0 0

Commit message: move_arm_complite

File: urdf_publisher/urdf/humanSubject01_48dof.urdf (robot description, URDF)
Before this commit: robot XSensStyleModel_template, 52 links, 51 joints
Links:
- added link LeftForeArm_f, mass 0
- added link LeftForeArm_f2, mass 0
Joints:
- added joint jLeftElbow_base: type fixed, parent LeftUpperArm, child LeftForeArm_f, origin xyz=0     0.26994           0 rpy=0 0 0
- added joint jLeftElbow_rotx: type revolute, parent LeftForeArm_f, child LeftForeArm_f1, origin xyz=0     0           0 rpy=0 0 0, axis 1 0 0, limit lower=-5 upper=5 effort=30 velocity=1.0
- joint jLeftElbow_roty: child LeftForeArm_f1 -> LeftForeArm_f2; limit lower=-1.5708 upper=1.48353 effort=30 velocity=1.0 -> lower=-5 upper=5 effort=30 velocity=1.0; origin xyz=0     0.26994           0 rpy=0 0 0 -> xyz=0 0 0 rpy=0 0 0; parent LeftUpperArm -> LeftForeArm_f1
- joint jLeftElbow_rotz: limit lower=-2.53073 upper=0 effort=30 velocity=1.0 -> lower=-5 upper=5 effort=30 velocity=1.0; parent LeftForeArm_f1 -> LeftForeArm_f2
- joint jLeftShoulder_rotx: limit lower=-1.5708 upper=2.35619 effort=30 velocity=1.0 -> lower=-5 upper=5 effort=30 velocity=1.0
- joint jLeftShoulder_roty: limit lower=-1.5708 upper=1.5708 effort=30 velocity=1.0 -> lower=-5 upper=5 effort=30 velocity=1.0
- joint jLeftShoulder_rotz: limit lower=-3.14159 upper=0.785398 effort=30 velocity=1.0 -> lower=-5 upper=5 effort=30 velocity=1.0
